File: frontPanel_100mm/frontPanel_100mm.kicad_pcb (KiCad board)
At the start: 2 copper layers, 93.5 x 43.2 mm, 24 parts, among them J1 Conn_02x25_Odd_Even, J10 ANALOG IN PORT 2, J11 ATO PORT 2, J12 PWM PORT 3, J13 ANALOG OUT 3, J14 I2C PORT 1, J15 1 WIRE PORT 1, J16 I2C PORT 2, J17 1 WIRE PORT 2, J2 GPIO PORT A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

Commit message: card edge revision
Parts:
- moved J1 2.64 mm to (146.8, 88.5)
Routing:
- net GND: track 137.5 -> 250.9 mm, vias 10 -> 15
- net /PA7: track 84.2 -> 40.4 mm, vias 0 -> 2
- net /PA5: track 75.8 -> 33.4 mm
- net /PA2: track 36.7 -> 77.3 mm
- net /PA6: track 70.5 -> 39.0 mm
- net /PA3: track 73.4 -> 43.2 mm, vias 0 -> 2
- net /PA8: track 72.3 -> 46.1 mm, vias 0 -> 1
- net /AIN4: track 42.1 -> 54.6 mm
- net /SDA: track 65.1 -> 54.6 mm, vias 0 -> 2
- net /AOUT4: track 51.3 -> 61.8 mm, vias 0 -> 1
- net /PA1: track 33.3 -> 42.3 mm, vias 0 -> 2
- net /AIN3: track 57.6 -> 65.6 mm
- net /AOUT8: track 65.1 -> 60.6 mm
- net /PA4: track 68.7 -> 73.1 mm
- net /AOUT2: track 71.4 -> 75.1 mm
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Other:
- net class Default: clearance 0.2 -> 0.15
- rule trace_clearance: 0.2 -> 0.15

Commit message: Tweak front panel size
Routing:
- net GND: track 250.9 -> 249.6 mm
- net /3v3: track 370.8 -> 370.0 mm
Other:
- board size 93.5 x 43.2 mm -> 92.9 x 44.3 mm
Changed lines of the file:
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@@
     (thickness 1.6)
     (drawings 89)
-    (tracks 666)
+    (tracks 665)
     (zones 0)
     (modules 24)
@@
     (effects (font (size 1 1) (thickness 0.15)) (justify left mirror))
   )
-  (gr_arc (start 192.43 92.18) (end 192.43 93.25) (angle -90) (layer Edge.Cuts) (width 0.01))
-  (gr_arc (start 101.07 92.18) (end 100 92.18) (angle -90) (layer Edge.Cuts) (width 0.01))
-  (gr_arc (start 101.07 51.07) (end 101.07 50) (angle -90) (layer Edge.Cuts) (width 0.01))
-  (gr_arc (start 192.43 51.07) (end 193.5 51.07) (angle -90) (layer Edge.Cuts) (width 0.01))
+  (gr_arc (start 192.13 92.18) (end 192.13 93.25) (angle -90) (layer Edge.Cuts) (width 0.01))
+  (gr_arc (start 101.37 92.18) (end 100.3 92.18) (angle -90) (layer Edge.Cuts) (width 0.01))
+  (gr_arc (start 101.37 50.07) (end 101.37 49) (angle -90) (layer Edge.Cuts) (width 0.01))
+  (gr_arc (start 192.13 50.07) (end 193.2 50.07) (angle -90) (layer Edge.Cuts) (width 0.01))
   (gr_line (start 105 88.25) (end 188.5 88.25) (layer Margin) (width 0.2))
   (gr_line (start 105 55) (end 188.5 55) (layer Margin) (width 0.2))
   (gr_line (start 188.5 55) (end 188.5 88.25) (layer Margin) (width 0.2))
   (gr_line (start 105 55) (end 105 88.25) (layer Margin) (width 0.2))
-  (gr_line (start 100 51.07) (end 100 92.18) (layer Edge.Cuts) (width 0.01))
-  (gr_line (start 193.5 51.05) (end 193.5 92.18) (layer Edge.Cuts) (width 0.01))
-  (gr_line (start 101.07 93.25) (end 192.43 93.25) (layer Edge.Cuts) (width 0.01))
-  (gr_line (start 101.04 50) (end 192.45 50) (layer Edge.Cuts) (width 0.01))
-  (segment (start 178.53 90.95) (end 180.05 90.95) (width 0.25) (layer F.Cu) (net 18))
-  (segment (start 178.41 85.95) (end 180.18 85.95) (width 0.25) (layer F.Cu) (net 18))
-  (segment (start 178.5 85.95) (end 180.96 85.95) (width 0.25) (layer B.Cu) (net 18))
-  (segment (start 101.42 92.39) (end 100.61 91.58) (width 0.25) (layer F.Cu) (net 1))
-  (segment (start 100.61 91.58) (end 100.61 51.8) (width 0.25) (layer F.Cu) (net 1))
-  (segment (start 100.61 51.8) (end 101.76 50.65) (width 0.25) (layer F.Cu) (net 1))
+  (gr_line (start 100.3 50.07) (end 100.3 92.18) (layer Edge.Cuts) (width 0.01))
+  (gr_line (start 193.2 50.07) (end 193.2 92.18) (layer Edge.Cuts) (width 0.01))
+  (gr_line (start 101.37 93.25) (end 192.13 93.25) (layer Edge.Cuts) (width 0.01))
+  (gr_line (start 101.37 49) (end 192.13 49) (layer Edge.Cuts) (width 0.01))
+  (segment (start 177.39 90.99) (end 179.42 90.99) (width 0.25) (layer F.Cu) (net 18))
+  (segment (start 177.53 85.92) (end 179.41 85.92) (width 0.25) (layer F.Cu) (net 18))
   (segment (start 106.84 52.75) (end 105.94 52.75) (width 0.25) (layer B.Cu) (net 1))
   (via (at 105.01 51.39) (size 0.8) (drill 0.4) (layers F.Cu B.Cu) (net 1))
@@
   (segment (start 105.01 51.82) (end 105.01 51.39) (width 0.25) (layer B.Cu) (net 1))
   (segment (start 105.01 51.39) (end 105.01 50.65) (width 0.25) (layer F.Cu) (net 1))
-  (segment (start 101.76 50.65) (end 105.01 50.65) (width 0.25) (layer F.Cu) (net 1))
   (segment (start 105.01 50.65) (end 166.41 50.65) (width 0.25) (layer F.Cu) (net 1))
   (segment (start 180.48 78.84) (end 180.48 67.995) (width 0.25) (layer B.Cu) (net 1))
@@
   (via (at 113.4 92.39) (size 0.8) (drill 0.4) (layers F.Cu B.Cu) (net 1))
   (segment (start 116.84 92.39) (end 113.4 92.39) (width 0.25) (layer F.Cu) (net 1))
-  (segment (start 113.4 92.39) (end 101.42 92.39) (width 0.25) (layer F.Cu) (net 1))
   (segment (start 180.48 67.995) (end 179.845 67.995) (width 0.25) (layer F.Cu) (net 1))
   (segment (start 179.845 67.995) (end 178.46 66.61) (width 0.25) (layer F.Cu) (net 1))
@@
   (segment (start 114.85 92.39) (end 116.27 90.97) (width 0.25) (layer B.Cu) (net 1))
   (segment (start 113.4 92.39) (end 114.85 92.39) (width 0.25) (layer B.Cu) (net 1))
+  (segment (start 102.13 50.65) (end 105.01 50.65) (width 0.25) (layer F.Cu) (net 1))
+  (segment (start 101.01 51.77) (end 102.13 50.65) (width 0.25) (layer F.Cu) (net 1))
+  (segment (start 101.01 91.57) (end 101.01 51.77) (width 0.25) (layer F.Cu) (net 1))
+  (segment (start 101.83 92.39) (end 101.01 91.57) (width 0.25) (layer F.Cu) (net 1))
+  (segment (start 113.4 92.39) (end 101.83 92.39) (width 0.25) (layer F.Cu) (net 1))
   (segment (start 154.048 78.84) (end 154.048 76.368) (width 0.25) (layer B.Cu) (net 2))
   (via (at 114.76 70.82) (size 0.8) (drill 0.4) (layers F.Cu B.Cu) (net 2))
@@
   (segment (start 176.615 89.085) (end 178.5 90.97) (width 0.25) (layer F.Cu) (net 18))
   (segment (start 148.29 89.085) (end 176.615 89.085) (width 0.25) (layer F.Cu) (net 18))
-  (segment (start 148.29 87.815) (end 148.29 88.41) (width 0.25) (layer B.Cu) (net 18))
-  (segment (start 148.29 88.41) (end 148.29 89.085) (width 0.25) (layer B.Cu) (net 18))
-  (segment (start 148.3 88.42) (end 150.99 88.42) (width 0.25) (layer B.Cu) (net 18))
-  (segment (start 177.33 90.94) (end 179.87 90.94) (width 0.25) (layer B.Cu) (net 18))
+  (segment (start 148.29 89.085) (end 148.29 87.815) (width 0.25) (layer B.Cu) (net 18))
+  (segment (start 148.3 88.47) (end 150.25 88.47) (width 0.25) (layer B.Cu) (net 18))
+  (segment (start 176.76 90.97) (end 178.65 90.97) (width 0.25) (layer B.Cu) (net 18))
+  (segment (start 178.49 85.91) (end 180.43 85.91) (width 0.25) (layer B.Cu) (net 18))
   (segment (start 151.83 89.92) (end 151.83 90.97) (width 0.25) (layer B.Cu) (net 18))
   (segment (start 150.995 89.085) (end 151.83 89.92) (width 0.25) (layer B.Cu) (net 18))
